File: MCU.kicad_sch (KiCad schematic)
At the start: 0 parts

Commit message: WIP
Parts:
- added U?: ATxmega128A1U-A, Package_QFP:TQFP-100_14x14mm_P0.5mm, symbol MCU_Microchip_ATmega:ATxmega128A1U-A
Connections:
- new net: U?.13 (GND), U?.23 (GND), U?.3 (GND), U?.33 (GND), U?.43 (GND), U?.53 (GND), U?.63 (GND), U?.73 (GND), U?.84 (GND), U?.93 (GND)
- new net: U?.14 (VCC), U?.24 (VCC), U?.34 (VCC), U?.44 (VCC), U?.54 (VCC), U?.64 (VCC), U?.74 (VCC), U?.83 (VCC)
- new net: U?.4 (AVCC), U?.94 (AVCC)
Changed lines of the file:
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@@
 (kicad_sch (version 20211123) (generator eeschema)
-  (paper "A4")
+  (paper "A3")
+  (hierarchical_label "SDA1" (shape bidirectional) (at 279.4 91.44 0)
+    (effects (font (size 1.27 1.27)) (justify left))
+  )
+  (hierarchical_label "SCL1" (shape bidirectional) (at 279.4 97.79 0)
+    (effects (font (size 1.27 1.27)) (justify left))
+  )
+  (hierarchical_label "SCL2" (shape bidirectional) (at 279.4 110.49 0)
+    (effects (font (size 1.27 1.27)) (justify left))
+  )
+  (hierarchical_label "SDA2" (shape bidirectional) (at 279.4 104.14 0)
+    (effects (font (size 1.27 1.27)) (justify left))
+  )
+  (symbol (lib_id "MCU_Microchip_ATmega:ATxmega128A1U-A") (at 154.94 97.79 0) (unit 1)
+    (in_bom yes) (on_board yes) (fields_autoplaced)
+    (property "Reference" "U?" (id 0) (at 156.9594 162.56 0)
+      (effects (font (size 1.27 1.27)) (justify left))
+    )
+    (property "Value" "ATxmega128A1U-A" (id 1) (at 156.9594 165.1 0)
+      (effects (font (size 1.27 1.27)) (justify left))
+    )
+    (property "Footprint" "Package_QFP:TQFP-100_14x14mm_P0.5mm" (id 2) (at 154.94 97.79 0)
+      (effects (font (size 1.27 1.27) italic) hide)
+    )
+    (property "Datasheet" "http://ww1.microchip.com/downloads/en/DeviceDoc/Atmel-8385-8-and-16-bit-AVR-Microcontroller-ATxmega64A1U-ATxmega128A1U_datasheet.pdf" (id 3) (at 154.94 97.79 0)
+      (effects (font (size 1.27 1.27)) hide)
+    )
+    (pin "1")
+    (pin "10")
+    (pin "100")
+    (pin "11")
+    (pin "12")
+    (pin "13")
+    (pin "14")
+    (pin "15")
+    (pin "16")
+    (pin "17")
+    (pin "18")
+    (pin "19")
+    (pin "2")
+    (pin "20")
+    (pin "21")
+    (pin "22")
+    (pin "23")
+    (pin "24")
+    (pin "25")
+    (pin "26")
+    (pin "27")
+    (pin "28")
+    (pin "29")
+    (pin "3")
+    (pin "30")
+    (pin "31")
+    (pin "32")
+    (pin "33")
+    (pin "34")
+    (pin "35")
+    (pin "36")
+    (pin "37")
+    (pin "38")
+    (pin "39")
+    (pin "4")
+    (pin "40")
+    (pin "41")
+    (pin "42")
+    (pin "43")
+    (pin "44")
+    (pin "45")
+    (pin "46")
+    (pin "47")
+    (pin "48")
+    (pin "49")
+    (pin "5")
+    (pin "50")
+    (pin "51")
+    (pin "52")
+    (pin "53")
+    (pin "54")
+    (pin "55")
+    (pin "56")
+    (pin "57")
+    (pin "58")
+    (pin "59")
+    (pin "6")
+    (pin "60")
+    (pin "61")
+    (pin "62")
+    (pin "63")
+    (pin "64")
+    (pin "65")
+    (pin "66")
+    (pin "67")
+    (pin "68")
+    (pin "69")
+    (pin "7")
+    (pin "70")
+    (pin "71")
+    (pin "72")
+    (pin "73")
+    (pin "74")
+    (pin "75")
+    (pin "76")
+    (pin "77")
+    (pin "78")
+    (pin "79")
+    (pin "8")
+    (pin "80")
+    (pin "81")
+    (pin "82")
+    (pin "83")
+    (pin "84")
+    (pin "85")
+    (pin "86")
+    (pin "87")
+    (pin "88")
+    (pin "89")
+    (pin "9")
+    (pin "90")
+    (pin "91")
+    (pin "92")
+    (pin "93")
+    (pin "94")
+    (pin "95")
+    (pin "96")
+    (pin "97")
+    (pin "98")
+    (pin "99")
+  )
 )
