File: tuner-scanner.kicad_sch (KiCad schematic)
At the start: 26 parts, among them U1 R820T2, U2 R828D

Commit message: WIP
Parts:
- C1, C2, C3, C4, C5, C6, C7, C8: renamed from C?; footprint (none) -> Capacitor_SMD:C_0603_1608Metric
- C9: renamed from 100n; value C -> 100n; footprint (none) -> Capacitor_SMD:C_0603_1608Metric
- J2, J4: renamed from J?; footprint (none) -> Connector_Coaxial:U.FL_Hirose_U.FL-R-SMT-1_Vertical
- L1, L2, L3, L4: renamed from L?; footprint (none) -> Inductor_SMD:L_0603_1608Metric
- R1: renamed from R?; footprint (none) -> Resistor_SMD:R_0612_1632Metric
- T1: renamed from T?; footprint TXF453229NF351 -> Samacsys:TXF453229NF351
- gave numbers to parts that had none: 5

Commit message: WIP
Parts:
- removed J4: Conn_Coaxial, Connector_Coaxial:U.FL_Hirose_U.FL-R-SMT-1_Vertical, symbol Connector:Conn_Coaxial
- removed U1: R820T2, Package_DFN_QFN:QFN-24-1EP_4x4mm_P0.5mm_EP2.15x2.15mm, symbol tuner:R820T2
- added U? (x4): LM2902, symbol Amplifier_Operational:LM2902
- renumbered C9 to C6, C6 to C7, C7 to C8, C8 to C9, J5 to J4, U2 to U1
Connections:
- net at C3.1, U1.8 (det2): now also U?.3 (+)
- net at C8.1, C9.1, U1.20 (CP): now also U?.10 (+)
- net at C2.1, U1.7 (det1): now also U?.5 (+)
- new net: U?.6 (-), U?.7
- new net: U?.1, U?.2 (-)
- new net: U?.8, U?.9 (-)
Other:
- removed sheet Untitled Sheet
- added sheet Tuner1 (Tuner1.kicad_sch)
- added sheet Tuner2 (Tuner1.kicad_sch)
- added sheet upmix (upmix.kicad_sch)
- sheet MCU: file untitled.kicad_sch -> MCU.kicad_sch
- sheet MCU ports: added SCL1, SCL2, SDA1, SDA2; removed none
